Commit message: Teleop Issue Resolved

File: washroom_cleaner/urdf/bot_base.urdf.xacro (robot description, xacro)
@@ -508,12 +508,27 @@
         <leftRearJoint>left_rear_wheel_joint</leftRearJoint>
         <rightRearJoint>right_rear_wheel_joint</rightRearJoint>
-        <wheelSeparation>0.71</wheelSeparation>
-        <wheelDiameter>0.215</wheelDiameter>
+        <wheelSeparation>0.79</wheelSeparation>
+        <wheelDiameter>0.18</wheelDiameter>
         <robotBaseFrame>base_link</robotBaseFrame>
-        <torque>1</torque>
+        <torque>5</torque>
         <topicName>cmd_vel</topicName>
         <broadcastTF>false</broadcastTF>
      </plugin>
     </gazebo>
+    <gazebo>
+      <plugin name="gazebo_ros_control" filename="libgazebo_ros_control.so">
+        <robotNamespace>/washroom_cleaner</robotNamespace>
+      </plugin>
+    </gazebo>
+    <transmission name="tran1">
+      <type>transmission_interface/SimpleTransmission</type>
+      <joint name="dustbin_joint">
+        <hardwareInterface>EffortJointInterface</hardwareInterface>
+      </joint>
+      <actuator name="motor1">
+        <hardwareInterface>EffortJointInterface</hardwareInterface>
+        <mechanicalReduction>1</mechanicalReduction>
+      </actuator>
+    </transmission>
   </xacro:macro>
 </robot>
